File: myStrava.sch (EAGLE design)
At the start: 27 parts, among them U1 ADXL345, U2 MAX1704X, U3 BMP180, U4 GTK

Commit message: Premiere board complete, manque l'ecran !
Parts:
- removed U1: ADXL345, SparkFun-Sensors:ADXL345
- added POLO: (no value), SparkFun-Connectors:M03LOCK
Connections:
- removed net N$3: U$1.CLK, U$2.13/SCK/LED, U1.SCL
- new net N$25: U$1.MOSI, U$2.12/MISO
- net GND: no longer U$2.AGND, U1.GND@2, U1.GND@4, U1.GND@5
- net GND-ISO: now also POLO.2, U$2.AGND
- net N$1: no longer U1.SDO
- net N$19: now also SWITCH.2; no longer R3.1, R4.1, SWITCH.3
- net N$2: now also POLO.1, R3.1, R4.1, SWITCH.3; no longer U$1.MOSI, U$2.12/MISO, U1.SDA
- net N$6: now also U$1.CLK, U$2.13/SCK/LED; no longer U$2.15/A1/T, U1.CS
- net V+: now also POLO.3; no longer SWITCH.2
- net VCC: no longer U1.VDD, U1.VS
Other:
- moved on the sheet: BATT, SWITCH

Commit message: Bare metal !!!
Parts:
- removed MCP: MCP73831, BaseApp:MCP73831
- removed POLO: (no value), SparkFun-Connectors:M03LOCK
- removed U$1: DM3AT, HIROSE-DM3AT:DM3AT
- removed U$10: ANTAP28, ANTAP28:ANTAP28
- removed U$2: TEENSY_3.1+4, Teensy_3_Series_Board_v1.0:TEENSY_3.1+4
- removed U$25: NAV_SWITCHSMD, SparkFun-Electromechanical:NAV_SWITCHSMD
- removed U2: MAX1704X, SparkFun-PowerIC:MAX1704X
- removed U3: BMP180, SparkFun-Sensors:BMP180
- removed U4: GTK, adafruit:GPS_FGPMMOPA6H
- added BMP180: BMP180, SparkFun-Sensors:BMP180
- added C10, C11, C9: 0.1uF, microbuilder:CAP_CERAMIC1206
- added JTAG: 2X5_0.05"_CORTEX_DEBUGTH_NOKEY_UNSHROUDED, con-cortex:2X5_0.05"_CORTEX_DEBUGTH_NOKEY_UNSHROUDED
- added LDO33: 3.3V/150mA, SparkFun-PowerIC:V_REG_MIC52053.3V
- added MAX17043: MAX1704X, SparkFun-PowerIC:MAX1704X
- added MCP73831: MCP73831, BaseApp:MCP73831
- added MK20DN512: MK20DN512, MK20DN512:MK20DN512
- added MT3339: GTK, adafruit:GPS_FGPMMOPA6H
- added N550: ANTAP28, ANTAP28:ANTAP28
- added NAV: NAV_SWITCHSMD, SparkFun-Electromechanical:NAV_SWITCHSMD
- added R10, R11, R12, R13, R14: 10k, SparkFun-Resistors:RESISTOR1206
- added R8, R9: 33ohm, SparkFun-Resistors:RESISTOR1206
- added SD: DM3AT, HIROSE-DM3AT:DM3AT
- added SHARP: SHARP27, sharp:SHARP27
- added SST25: FLASH, FlashMem:FLASH
- added USB: USB-MICROB, SparkFun-Connectors:USB-MICROB
- added Y1: 16MHz, SparkFun-FreqCtrl:CRYSTALHC49UV
- C2, C3, C6: device SparkFun-Capacitors:CAP_POL1206 -> microbuilder:CAP_CERAMIC1206
- SWITCH: value (none) -> NAVI
Connections:
- removed net GND-ISO: BATT.2, C1.1, C4.2, C5.2, MCP.VSS, POLO.2, R1.1, R7.2, U$2.AGND, U2.CTG, U2.GND@4, U2.GND@EP
- removed net N$10: U$2.8/TX3, U4.RX
- removed net N$11: U$10.SUSPEND, U$2.17/A3/T
- removed net N$12: U$10.SLEEP, U$2.21/A7/PWM
- removed net N$13: U$10.RST, U$2.23/A9/T/PWM
- removed net N$15: U$10.RX, U$2.10/TX2/PWM
- removed net N$24: U$2.22/A8/T/PWM, U$25.1
- removed net N$5: U$1.CS, U$2.2
- removed net N$6: U$1.CLK, U$2.13/SCK/LED
- removed net N$9: U$2.7/RX3, U4.TX
- removed net SCL: R5.2, U$2.19/A5/T/SCL0, U2.SCL, U3.SCL
- removed net SDA: R6.2, U$2.18/A4/T/SDA0, U2.SDA, U3.SDA
- removed net V+: POLO.3, U$2.VIN
- removed net VCC: C2.+, C3.+, C6.+, C7.P$1, C8.P$1, R5.1, R6.1, U$1.VCC, U$10.VCC, U$2.3.3V, U3.VDD, U3.VDDIO, U4.VCC
- new net MK_DI: MK20DN512.PTC7, SD.MISO, SST25.SO
- new net MK_DO: MK20DN512.PTC6, SD.MOSI, SHARP.MOSI, SST25.SI
- new net MK_RX1: MK20DN512.PTB16, MT3339.TX
- new net MK_RX3: MK20DN512.PTD2, N550.TX
- new net MK_SCL: BMP180.SCL, MAX17043.SCL, MK20DN512.PTB2, R5.2
- new net MK_SCLK: MK20DN512.PTC5, SD.CLK, SHARP.SCLK, SST25.SCK
- new net MK_SDA: BMP180.SDA, MAX17043.SDA, MK20DN512.PTB3, R6.2
- new net MK_TX1: MK20DN512.PTB17, MT3339.RX
- new net MK_TX3: MK20DN512.PTD3, N550.RX
- new net N$26: R11.1, SHARP.EXTCOMM
- new net N$27: C11.P$1, R12.1, SHARP.DISP
- new net N$29: MK20DN512.PTB18, NAV.2
- new net N$30: MK20DN512.PTB19, NAV.T
- new net N$31: MK20DN512.PTB0, NAV.1
- new net N$32: MK20DN512.PTC0, SST25.CE
- new net N$33: R14.1, SST25.WP
- new net N$34: R13.2, SST25.HOLD
- new net N$35: JTAG.~RESET, MK20DN512.RESET
- new net TCLK: JTAG.SWDCLK/TCK, MK20DN512.PTA0
- new net TDI: JTAG.NC/TDI, MK20DN512.PTA1
- new net TDO: JTAG.SWO/TDO, MK20DN512.PTA2
- new net TMS: JTAG.SWDIO/TMS, MK20DN512.PTA3
- new net USB1_DM_N: R9.1, USB.D-
- new net USB1_DP_P: R8.1, USB.D+
- new net USB_DM_N: MK20DN512.USB0_DM, R9.2
- new net USB_DP_P: MK20DN512.USB0_DP, R8.2
- new net VCC-ISO: LDO33.EN, LDO33.IN, R3.1, R4.1, SWITCH.3
- new net VDD: BMP180.VDD, BMP180.VDDIO, C2.P$1, C3.P$1, C6.P$1, C7.P$1, C8.P$1, C9.P$1, JTAG.VCC, LDO33.OUT, MK20DN512.VBAT, MK20DN512.VDD, MK20DN512.VDD1, MK20DN512.VDD2, MK20DN512.VDD3, MK20DN512.VDD4, MK20DN512.VDD5, MK20DN512.VDDA, MK20DN512.VOUT33, MK20DN512.VREFH, MT3339.VCC, N550.VCC, R12.2, R13.1, R14.2, R5.1, R6.1, SD.VCC, SHARP.VDD, SHARP.VDDA, SST25.VDD
- net GND: now also BATT.2, BMP180.GND, C1.1, C10.P$2, C11.P$2, C2.P$2, C3.P$2, C4.2, C5.2, C6.P$2, C9.P$2, JTAG.GND, JTAG.GND-DETECT, LDO33.GND, MAX17043.CTG, MAX17043.GND@4, MAX17043.GND@EP, MCP73831.VSS, MK20DN512.VREFL, MK20DN512.VSS, MK20DN512.VSS1, MK20DN512.VSS2, MK20DN512.VSS3, MK20DN512.VSS4, MK20DN512.VSS5, MK20DN512.VSSA, MT3339.GND@1, MT3339.GND@2, MT3339.GND@3, MT3339.GND@4, N550.GND, N550.GND2, NAV.C, R1.1, R10.1, R11.2, R7.2, SD.GND, SHARP.VSS, SHARP.VSSA, SST25.VSS, USB.GND; no longer C2.-, C3.-, C6.-, U$1.GND, U$10.BR1, U$10.GND, U$10.GND2, U$10.NONE3, U$10.PORTSEL, U$10.SCLK, U$10.SPD_SEL, U$2.GND, U$25.C, U3.GND, U4.GND@1, U4.GND@2, U4.GND@3, U4.GND@4
- net N$1: now also MK20DN512.PTC1, SD.CS; no longer U$1.MISO, U$2.11/MOSI
- net N$14: now also MK20DN512.PTA19, Y1.2; no longer U$10.BOOT, U$2.5/PWM
- net N$16: now also MCP73831.PROG; no longer MCP.PROG
- net N$17: now also MCP73831.STAT; no longer MCP.STAT
- net N$18: now also MCP73831.VDD, USB.VBUS; no longer MCP.VDD, U$2.VUSB
- net N$19: now also MK20DN512.PTA18, Y1.1; no longer BATT.1, C5.1, MCP.VBAT, SWITCH.2
- net N$2: now also BATT.1, C5.1, MCP73831.VBAT, SWITCH.2; no longer POLO.1, R3.1, R4.1, SWITCH.3
- net N$21: now also MK20DN512.PTD4, N550.BR1; no longer U$10.TX, U$2.9/RX2/PWM
- net N$22: now also MK20DN512.PTC2, SHARP.CS; no longer U$2.14/A0, U$25.2
- net N$23: now also C10.P$1, MK20DN512.VREF_OUT; no longer U$2.16/A2/T, U$25.T
- net N$25: now also R10.2, SHARP.EXTMODE; no longer U$1.MOSI, U$2.12/MISO
- net N$4: now also MAX17043.CELL; no longer U2.CELL
- net N$7: now also MAX17043.VDD; no longer U2.VDD
- net N$8: now also MAX17043.QST; no longer U2.QST
Other:
- moved on the sheet: BATT, C1, C4, C5, C7, C8, D1, R1, R2, R3, R4, R5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

Commit message: Routage initial
Parts:
- added SPK: FARNELL_SPK, Strutz Electronic Industries:MDMK2020T4R7MM
Connections:
- net USB1_DP_P renamed USB1_DM_P
- net USB_DP_P renamed USB_DM_P
- new net N$3: MK20DN512.PTB1, SPK.1
- net GND: now also SPK.2
Changed lines of the file:
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@@
 <clearance class="2" value="0.1524"/>
 </class>
-<class number="3" name="usb" width="0.254" drill="0.1524">
-<clearance class="3" value="0.1524"/>
+<class number="3" name="usb" width="0.2032" drill="0.1524">
+<clearance class="0" value="0.1524"/>
+<clearance class="1" value="0.1524"/>
+<clearance class="2" value="0.1524"/>
+<clearance class="3" value="0.2286"/>
 </class>
 </classes>
@@
 <part name="U$51" library="microbuilder" deviceset="GND" device=""/>
 <part name="SUPPLY19" library="supply2" deviceset="VCC" device=""/>
+<part name="U$2" library="microbuilder" deviceset="GND" device=""/>
+<part name="SPK" library="Strutz Electronic Industries" deviceset="MDMK2020T4R7MM" device="" value="FARNELL_SPK"/>
 </parts>
 <sheets>
@@
 <instance part="U$51" gate="G$1" x="-40.64" y="-246.38" rot="R180"/>
 <instance part="SUPPLY19" gate="G$1" x="-22.86" y="-248.92"/>
+<instance part="U$2" gate="G$1" x="83.82" y="-193.04" rot="R90"/>
+<instance part="SPK" gate="G$1" x="66.04" y="-193.04"/>
 </instances>
 <busses>
@@
 <wire x1="-38.1" y1="-251.46" x2="-40.64" y2="-251.46" width="0.1524" layer="91"/>
 <junction x="-40.64" y="-251.46"/>
+</segment>
+<segment>
+<pinref part="SPK" gate="G$1" pin="2"/>
+<pinref part="U$2" gate="G$1" pin="GND"/>
+<wire x1="73.66" y1="-193.04" x2="81.28" y2="-193.04" width="0.1524" layer="91"/>
 </segment>
 </net>
@@
 </segment>
 </net>
-<net name="USB_DP_P" class="3">
+<net name="USB_DM_P" class="3">
 <segment>
 <pinref part="R8" gate="G$1" pin="2"/>
@@
 </segment>
 </net>
-<net name="USB1_DP_P" class="3">
+<net name="USB1_DM_P" class="3">
 <segment>
 <pinref part="USB" gate="G$1" pin="D+"/>
@@
 </segment>
 </net>
+<net name="N$3" class="0">
+<segment>
+<pinref part="MK20DN512" gate="G$1" pin="PTB1"/>
+<pinref part="SPK" gate="G$1" pin="1"/>
+<wire x1="45.72" y1="-193.04" x2="58.42" y2="-193.04" width="0.1524" layer="91"/>
+</segment>
+</net>

Commit message: Candidat V2
Parts:
- removed N550: ANTAP28, ANTAP28:ANTAP28
- added JTAG1: 2X5_0.05"_CORTEX_DEBUGTH_NOKEY_UNSHROUDED, con-cortex:2X5_0.05"_CORTEX_DEBUGTH_NOKEY_UNSHROUDED
- added LED1: (no value), adafruit:LEDCHIPLED_1206
- added R15: 180, SparkFun-Resistors:RESISTOR1206
- added U$1: N548, N548:N548
- added U$17: GPS_TX, Exposed_pad:MDMK2020T4R7MM
- added U$26: PTE0, Exposed_pad:MDMK2020T4R7MM
- added U$32: PTE1, Exposed_pad:MDMK2020T4R7MM
- R8, R9: device SparkFun-Resistors:RESISTOR1206 -> SparkFun-Resistors:RESISTOR0805-RES
Connections:
- removed net MK_RX3: MK20DN512.PTD2, N550.TX
- removed net MK_TX3: MK20DN512.PTD3, N550.RX
- removed net VDD: BMP180.VDD, BMP180.VDDIO, C2.P$1, C3.P$1, C6.P$1, C7.P$1, C8.P$1, C9.P$1, JTAG.VCC, LDO33.OUT, MK20DN512.VBAT, MK20DN512.VDD, MK20DN512.VDD1, MK20DN512.VDD2, MK20DN512.VDD3, MK20DN512.VDD4, MK20DN512.VDD5, MK20DN512.VDDA, MK20DN512.VOUT33, MK20DN512.VREFH, MT3339.VCC, N550.VCC, R12.2, R13.1, R14.2, R5.1, R6.1, SD.VCC, SHARP.VDD, SHARP.VDDA, SST25.VDD
- new net N$10: SPK.2, U$1.P002
- new net N$11: MK20DN512.PTD3, U$1.P005
- new net N$12: MK20DN512.PTD2, U$1.P009
- new net N$13: MK20DN512.PTD4, U$1.P003
- new net N$15: MK20DN512.PTD5, U$1.P008
- new net N$24: MK20DN512.PTE1, U$32.1
- new net N$28: JTAG1.SWDIO/TMS, U$1.SWDIO
- new net N$5: NAV.T, U$1.P030
- new net N$6: NAV.1, U$1.P024
- new net N$9: NAV.C, U$1.P001
- new net VCC: BMP180.VDD, BMP180.VDDIO, C2.P$1, C3.P$1, C6.P$1, C7.P$1, C8.P$1, C9.P$1, JTAG.VCC, JTAG1.VCC, LDO33.OUT, MK20DN512.VBAT, MK20DN512.VDD, MK20DN512.VDD1, MK20DN512.VDD2, MK20DN512.VDD3, MK20DN512.VDD4, MK20DN512.VDD5, MK20DN512.VDDA, MK20DN512.VOUT33, MK20DN512.VREFH, MT3339.VCC, R12.2, R13.1, R14.2, R5.1, R6.1, SD.VCC, SHARP.VDD, SHARP.VDDA, SST25.VDD, U$1.VCC
- net GND: now also JTAG1.GND, JTAG1.GND-DETECT, R15.1, SPK.1, U$1.GND; no longer N550.GND, N550.GND2, NAV.C, SPK.2
- net MK_RX1: now also U$17.1
- net N$21: now also MK20DN512.PTE0, U$26.1; no longer MK20DN512.PTD4, N550.BR1
- net N$29: now also JTAG1.SWDCLK/TCK, U$1.SWDCLK; no longer MK20DN512.PTB18, NAV.2
- net N$3: now also NAV.2, U$1.P031; no longer MK20DN512.PTB1, SPK.1
- net N$30: now also LED1.A, MK20DN512.PTB1; no longer MK20DN512.PTB19, NAV.T
- net N$31: now also LED1.C, R15.2; no longer MK20DN512.PTB0, NAV.1
Other:
- moved on the sheet: NAV, SPK
